File: IC Design/Cabir_Control_Panel/Cabir_Control_Panel.kicad_pcb (KiCad board)
At the start: 2 copper layers, 80 x 41 mm, 24 parts

Commit message: Circuit design - initial
Parts:
- renumbered AC-DC1 to PS1
Changed lines of the file:
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@@
 		(layer "F.Cu")
 		(at 75.25 70.15)
-		(property "Reference" "AC-DC1"
+		(property "Reference" "PS1"
 			(at -12.95 5.5 90)
 			(unlocked yes)
